File: pcb/modelh.kicad_pcb (KiCad board)
At the start: 2 copper layers, 150 x 38 mm, 51 parts, among them J1 USB_B, J2 Conn_cols, J3 Conn_rows, J4 Conn_leds, J5 Conn_02x03_Odd_Even, J6 Conn_02x05_Odd_Even, J7 Conn_01x05, J8 Conn_01x05, J9 Conn_01x05, SW1 SW_Push, U1 STM32F103C8Tx, U2 AMS1117-3.3, Y1 8MHz

Commit message: v0.1
Parts:
- removed C1, C3: 10uF, Capacitor_SMD:C_0603_1608Metric
- removed C10, C11, C12, C13, C14, C2, C4, C9: 100nF, Capacitor_SMD:C_0402_1005Metric
- removed C5, C6: 20pF, Capacitor_SMD:C_0603_1608Metric
- removed the G*** at (150.2, 74.2)
- removed J5: Conn_02x03_Odd_Even, Connector_PinHeader_2.54mm:PinHeader_2x03_P2.54mm_Vertical
- removed J6: Conn_02x05_Odd_Even, Connector_IDC:IDC-Header_2x05_P2.54mm_Vertical
- removed J7, J8, J9: Conn_01x05, Connector_PinSocket_2.54mm:PinSocket_1x05_P2.54mm_Vertical
- removed LED1, LED2: green, LED_SMD:LED_0805_2012Metric
- removed R1, R2: 330, Resistor_SMD:R_0603_1608Metric
- removed R10, R11, R5: 1.5k, Resistor_SMD:R_0603_1608Metric
- removed R12, R13, R14, R15, R16: 0, Resistor_SMD:R_0805_2012Metric_Pad1.15x1.40mm_HandSolder
- removed R17, R18: 100k, Resistor_SMD:R_0603_1608Metric
- removed R3, R4: 22, Resistor_SMD:R_0603_1608Metric
- removed R6: 1M, Resistor_SMD:R_0603_1608Metric
- removed REF** (x2): MountingHole_4mm, MountingHole:MountingHole_4mm
- removed REF** (x2): MountingHole_3.5mm, MountingHole:MountingHole_3.5mm
- removed SW1: SW_Push, Button_Switch_SMD:SW_SPST_EVPBF
- removed TP1: TestPoint, TestPoint:TestPoint_THTPad_D1.5mm_Drill0.7mm
- removed Y1: 8MHz, Crystal:Crystal_SMD_5032-2Pin_5.0x3.2mm
- added G***: LOGO, Library:qr, F.Cu at (196.5, 63.7)
- added H1: Stand, MountingHole:MountingHole_4mm_Pad_Via, F.Cu at (209.8, 80.0)
- added H2: Stand, MountingHole:MountingHole_4mm_Pad_Via, F.Cu at (69.8, 72.0)
- added H3: Front, Library:Hole 3.5mm, F.Cu at (76.8, 52.0)
- added H4: Front, Library:Hole 3.5mm, F.Cu at (100.8, 52.0)
- added JP5: Reset jumper, Jumper:SolderJumper-2_P1.3mm_Open_RoundedPad1.0x1.5mm, F.Cu at (100.3, 58.3)
- added U3: 74HC595, PCM_Package_DIP_AKL:DIP-16_W7.62mm_Socket_LongPads, F.Cu at (129.3, 66.0)
- J1: value USB_B -> Battery Conn; footprint Connector_USB:USB_B_OST_USB-B1HSxx_Horizontal -> Connector_JST:JST_PH_S3B-PH-K_1x03_P2.00mm_Horizontal
- J2: value Conn_cols -> Conn_01x16; footprint modelh:ModelH-triomate-cols16 -> Library:ModelH-triomate-cols16
- J3: value Conn_rows -> Conn_01x12; footprint modelh:ModelH-triomate-rows12 -> Library:ModelH-triomate-rows12
- J4: value Conn_leds -> Conn_01x04; footprint modelh:ModelH-tripmate-leds4 -> Library:ModelH-triomate-leds4
- R7, R8, R9: footprint Resistor_SMD:R_0805_2012Metric -> Resistor_THT:R_Axial_DIN0207_L6.3mm_D2.5mm_P10.16mm_Horizontal
- U1: value STM32F103C8Tx -> nice_nano; footprint Package_QFP:LQFP-48_7x7mm_P0.5mm -> Library:nice_nano
- U2: value AMS1117-3.3 -> 74HC595; footprint Package_TO_SOT_SMD:SOT-223-3_TabPin2 -> PCM_Package_DIP_AKL:DIP-16_W7.62mm_Socket_LongPads
- moved R7 72.1 mm to (121.3, 79.7)
- moved R8 70.9 mm to (121.3, 76.5)
- moved R9 70.0 mm to (121.3, 73.3)
- moved J1 50.4 mm to (133.5, 78.0)
- moved U2 24.6 mm to (107.1, 66.2), turned to 90 degrees
- moved U1 19.5 mm to (88.8, 64.8), turned to 0 degrees
- moved J3 15.2 mm to (173.1, 50.0)
- moved J4 10.2 mm to (200.5, 51.0), turned to 0 degrees
- moved J2 5.49 mm to (130.3, 51.0)
Connections:
- J1 pad 1: Net-(J1-Pad1) -> GND
- J1 pad 2: Net-(J1-Pad2) -> +BATT
- J1 pad 3: Net-(J1-Pad3) -> GND
- J3 pad 10: Net-(J3-Pad10) -> +3.3V
- J3 pad 11: Net-(J3-Pad11) -> Net-(J3-Pin_11)
- J3 pad 12: Net-(J3-Pad12) -> Net-(J3-Pin_12)
- J3 pad 9: Net-(J3-Pad9) -> Net-(J3-Pin_9)
- J4 pad 1: Net-(J4-Pad1) -> Net-(J3-Pin_12)
- J4 pad 2: Net-(J4-Pad2) -> Net-(J3-Pin_11)
- J4 pad 3: +3V3 -> +3.3V
- J4 pad 4: Net-(J4-Pad4) -> Net-(J3-Pin_9)
- R7 pad 1: Net-(J4-Pad1) -> Net-(J3-Pin_12)
- R8 pad 1: Net-(J4-Pad2) -> Net-(J3-Pin_11)
- R9 pad 1: Net-(J4-Pad4) -> Net-(J3-Pin_9)
- U1 pad 10: row5 -> unconnected-(U1-100-Pad10)
- U1 pad 11: row7 -> led2
- U1 pad 12: row6 -> led1
- U1 pad 13: col15 -> led0
- U1 pad 15: col13 -> +BATT
- U1 pad 16: col12 -> GND
- U1 pad 17: col11 -> Net-(JP5-A)
- U1 pad 18: col10 -> +3.3V
- U1 pad 19: col9 -> row0
- U1 pad 2: STATUSLED -> SCLK
- U1 pad 20: BOOT1 -> row1
- U1 pad 21: col8 -> row2
- U1 pad 22: col7 -> row3
- U1 pad 23: GND -> row4
- U1 pad 24: +3V3 -> row5
- U1 pad 25: col6 -> row6
- U1 pad 26: col5 -> row7
- U1 pad 3: (no net) -> CS
- U1 pad 4: (no net) -> GND
- U1 pad 5: OSC8OUT -> GND
- U1 pad 6: OSC8IN -> MOSI
- U1 pad 7: nRST -> unconnected-(U1-020-Pad7)
- U1 pad 8: GND -> unconnected-(U1-022-Pad8)
- U1 pad 9: +3V3 -> unconnected-(U1-024-Pad9)
- U2 pad 1: GND -> col1
- U2 pad 2: +3V3 -> col2
- U2 pad 3: +5V -> col3
Routing:
- net +3V3: track 229.5 -> 0.00 mm, vias 4 -> 0
- net Net-(J3-Pin_9): track 0.00 -> 101.9 mm
- net Net-(J3-Pin_11): track 0.00 -> 94.1 mm
- net Net-(J3-Pin_12): track 0.00 -> 89.0 mm
- net +BATT: track 0.00 -> 80.8 mm
- net SCLK: track 0.00 -> 73.7 mm
- net CS: track 0.00 -> 71.0 mm
- net led0: track 98.3 -> 30.9 mm, vias 3 -> 0
- net led1: track 98.3 -> 31.1 mm, vias 3 -> 0
- net led2: track 98.4 -> 31.4 mm, vias 3 -> 0
- net nRST: track 46.2 -> 0.00 mm, vias 2 -> 0
- net MOSI: track 0.00 -> 35.4 mm
- net SWDIO: track 34.6 -> 0.00 mm, vias 2 -> 0
- net GND: track 31.3 -> 0.00 mm, vias 268 -> 0
- net SWCLK: track 29.9 -> 0.00 mm, vias 2 -> 0
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- added copper zone on B.Cu, net +3.3V
- added copper zone on In1.Cu, net GND
- added copper zone on In2.Cu, net GND
- removed copper zone on B.Cu, net GND
Other:
- copper layers 2 -> 4
- net class Default removed
- board text added: "54x28mm Reserved for Li-Po battery"
- board text added: "DOUBLE CHECK POLARITY"
- board text added: "Model K"
- board text added: "PWR"
- board text added: "Q/A"
- board text added: "RESET"
- board text added: "REVISION ${REVISION} ISSUED ${ISSUE_DATE}"
- board text added: "S/N"
- board text added: "https://rusz.space/modelk"
- board text removed: "3.3V"
- board text removed: "5V"
- board text removed: "Boot0"
- board text removed: "Boot1"
- board text removed: "Custom LED"
- board text removed: "Debug"
- board text removed: "LED0"
- board text removed: "LED1"
- board text removed: "LED2"
- board text removed: "Reset"
- board text removed: "https://modelh.club"
- board text removed: "v1.0a"
